File: pcb/R1000A.kicad_pcb (KiCad board)
At the start: 4 copper layers, 175 x 65.5 mm, 117 parts, among them J01 PCIESOCKET-X1, J02 PCIESOCKET-X1, J03 PCIESOCKET-X1, J04 PCIESOCKET-X1, J05 PCIESOCKET-X1, J06 PCIESOCKET-X1, J07 PCIESOCKET-X1, J08 PCIESOCKET-X1, J09 PCIESOCKET-X1, J10 PCIESOCKET-X1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

Commit message: layout wip
Connections:
- C13 pad 1: HT -> PFET_D
- C14 pad 1: HT -> PFET_D
- U3 pad 2: HT -> PFET_D
- U3 pad 3: HT -> PFET_D
Routing:
- net /PowerMonitor/IIN+: track 0.00 -> 121.3 mm, vias 0 -> 3
- net /PowerMonitor/IIN-: track 0.00 -> 120.2 mm, vias 0 -> 3
- net PFET_D: track 179.3 -> 287.7 mm, vias 22 -> 43
- net 5V0+: track 0.00 -> 86.2 mm, vias 0 -> 2
- net 5V0-: track 0.00 -> 83.4 mm, vias 0 -> 2
- net 3V3-: track 0.00 -> 33.2 mm, vias 0 -> 2
- net ~MRESET: track 301.6 -> 269.9 mm
- net +5V: track 14.0 -> 40.2 mm, vias 5 -> 10
- net 3V3+: track 0.00 -> 22.6 mm, vias 0 -> 2
- net HT: track 207.1 -> 224.6 mm, vias 26 -> 24
- net (no net): track 11.9 -> 0.18 mm, vias 14 -> 0
- net SCL0: track 226.8 -> 236.6 mm
- net +3V3: track 45.2 -> 53.6 mm, vias 21 -> 23
- net SDA0: track 210.2 -> 217.9 mm
- net /PowerMonitor/IN-2: track 0.00 -> 4.17 mm
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